Commit message: Updated box urdf

File: box_description/urdf/box.urdf.xacro (robot description, xacro)
@@ -1,7 +1,7 @@
 <?xml version="1.0"?>
 <robot name="box" xmlns:xacro="http://www.ros.org/wiki/xacro">
-<xacro:property name="box_len_x" value="0.25" />
-<xacro:property name="box_len_y" value="0.15" />
-<xacro:property name="box_len_z" value="0.08" />
+<xacro:property name="box_len_x" value="0.156" />
+<xacro:property name="box_len_y" value="0.257" />
+<xacro:property name="box_len_z" value="0.0794" />
 <xacro:property name="box_origin_from_corner" value="${box_len_x/2} ${box_len_y/2} ${box_len_z/2}" />
 <link name="box_base_link">
@@ -14,13 +14,16 @@
 <link name="box_center_link">
   <visual>
-    <origin rpy="0 0 0" xyz="0 0 0"/>
-    <geometry>
-      <mesh filename="package://box_description/meshes/box.dae"/>
-    </geometry>
+    <origin rpy="0 0 0" xyz="-${box_len_x/2} -${box_len_y/2} -${box_len_z/2}"/>
+    <geometry>
+      <mesh filename="file:///media/jos/ExternalSSD/thi_robothix_grand_challenge/box_description/meshes/box.dae" scale="0.001 0.001 0.001"/>
+    </geometry>
+    <material name="white">
+      <color rgba="1 1 1 1"/>
+    </material>
   </visual>
   <collision>
-    <origin rpy="0 0 0" xyz="0 0 0"/>
-    <geometry>
-      <box size="${box_len_x} ${box_len_y} ${box_len_z}"/>
+    <origin rpy="0 0 0" xyz="-${box_len_x/2} -${box_len_y/2} -${box_len_z/2}"/>
+    <geometry>
+      <box size="-${box_len_x/2} -${box_len_y/2} -${box_len_z/2}}"/>
     </geometry>
   </collision>
@@ -30,5 +33,5 @@
   <parent link="box_center_link"/>
   <child link="box_corner_1"/>
-  <origin rpy="0 0 0" xyz="${box_len_x/2} ${box_len_y/2} 0"/>
+  <origin rpy="0 0 0" xyz="-${box_len_x/2} -${box_len_y/2} -${box_len_z/2}"/>
 </joint>
 <link name="box_corner_1">
@@ -43,5 +46,5 @@
   <parent link="box_center_link"/>
   <child link="box_corner_2"/>
-  <origin rpy="0 0 0" xyz="${-1 * box_len_x/2} ${box_len_y/2} 0"/>
+  <origin rpy="0 0 0" xyz="${-1 * box_len_x/2} ${box_len_y/2} -${box_len_z/2}"/>
 </joint>
 <link name="box_corner_2">
@@ -56,5 +59,5 @@
   <parent link="box_center_link"/>
   <child link="box_corner_3"/>
-  <origin rpy="0 0 0" xyz="${box_len_x/2} ${-1 * box_len_y/2} 0"/>
+  <origin rpy="0 0 0" xyz="${box_len_x/2} ${box_len_y/2} -${box_len_z/2}"/>
 </joint>
 <link name="box_corner_3">
@@ -69,5 +72,5 @@
   <parent link="box_center_link"/>
   <child link="box_corner_4"/>
-  <origin rpy="0 0 0" xyz="${-1 * box_len_x/2} ${-1 * box_len_y/2} 0"/>
+  <origin rpy="0 0 0" xyz="${box_len_x/2} ${-1 * box_len_y/2} -${box_len_z/2}"/>
 </joint>
 <link name="box_corner_4">
@@ -81,40 +84,47 @@
 <!-- Buttons -->
 <joint name="box_button_blue_joint" type="fixed">
-  <parent link="box_base_link"/>
+  <parent link="box_corner_2"/>
   <child link="box_button_blue"/>
-  <origin rpy="0 0 0" xyz="0 0 ${box_len_z}"/>
+  <origin rpy="0 0 0" xyz="0.03405 -0.03225 ${box_len_z}"/>
 </joint>
 <link name="box_button_blue">
   <visual>
-    <origin rpy="0 0 0" xyz="0 0 0"/>
-    <geometry>
-      <cylinder radius="0.01" length="0.1"/>
-    </geometry>
+    <origin rpy="0 0 0" xyz="0 0 ${0.0041/2}"/>
+    <geometry>
+      <cylinder radius="0.00525" length="0.0041"/>
+    </geometry>
+    <material name="blue">
+      <color rgba="0 0 1 1"/>
+    </material>
   </visual>
 </link>
 <joint name="box_button_red_joint" type="fixed">
-  <parent link="box_base_link"/>
+  <parent link="box_corner_2"/>
   <child link="box_button_red"/>
-  <origin rpy="0 0 0" xyz="0 0 ${box_len_z}"/>
+  <origin rpy="0 0 0" xyz="0.04805 -0.03225 ${box_len_z}"/>
 </joint>
 <link name="box_button_red">
   <visual>
-    <origin rpy="0 0 0" xyz="0 0 0"/>
-    <geometry>
-      <cylinder radius="0.01" length="0.1"/>
-    </geometry>
+    <origin rpy="0 0 0" xyz="0 0 ${0.0041/2}"/>
+    <geometry>
+      <cylinder radius="0.00525" length="0.0041"/>
+    </geometry>
+    <material name="red">
+      <color rgba="1 0 0 1"/>
+    </material>
   </visual>
 </link>
 <!-- Slider -->
-<joint name="box_slider_joint" type="fixed">
-  <parent link="box_base_link"/>
+<joint name="box_slider_joint" type="prismatic">
+  <parent link="box_corner_3"/>
   <child link="box_slider"/>
-  <origin rpy="0 0 0" xyz="0 0 ${box_len_z}"/>
+  <origin rpy="0 0 0" xyz="-0.0425 -0.0675 ${box_len_z}"/>
+  <limit effort="1000.0" lower="-0.0215" upper="0.0215" velocity="0.5"/>
 </joint>
 <link name="box_slider">
   <visual>
-    <origin rpy="0 0 0" xyz="0 0 0"/>
-    <geometry>
-      <box size="0.03 0.01 0.01"/>
+    <origin rpy="0 0 0" xyz="0 0 0.005"/>
+    <geometry>
+      <box size="0.007 0.005796 0.01"/>
     </geometry>
   </visual>
@@ -122,49 +132,71 @@
 <!-- Sockets -->
 <joint name="box_socket_red_joint" type="fixed">
+  <parent link="box_corner_2"/>
+  <child link="box_socket_red"/>
+  <origin rpy="0 0 0" xyz="0.0589 -0.0895 ${box_len_z}"/>
+</joint>
+<link name="box_socket_red">
+  <visual>
+    <origin rpy="0 0 0" xyz="0 0 0.001"/>
+    <geometry>
+      <cylinder radius="0.007" length="0.002"/>
+    </geometry>
+    <material name="red">
+      <color rgba="1 0 0 1"/>
+    </material>
+  </visual>
+</link>
+<joint name="box_socket_black_joint" type="fixed">
+  <parent link="box_corner_2"/>
+  <child link="box_socket_black"/>
+  <origin rpy="0 0 0" xyz="0.034 -0.0895 ${box_len_z}"/>
+</joint>
+<link name="box_socket_black">
+  <visual>
+    <origin rpy="0 0 0" xyz="0 0 0.001"/>
+    <geometry>
+      <cylinder radius="0.007" length="0.002"/>
+    </geometry>
+    <material name="black">
+      <color rgba="0 0 0 1"/>
+    </material>
+  </visual>
+</link>
+<joint name="box_socket_grey_joint" type="fixed">
+  <parent link="box_corner_4"/>
+  <child link="box_socket_grey"/>
+  <origin rpy="0 -${pi/2} 0" xyz="-0.0482 0.0265 0.0963"/>
+</joint>
+<link name="box_socket_grey">
+  <visual>
+    <origin rpy="0 0 0" xyz="0 0 -0.001"/>
+    <geometry>
+      <cylinder radius="0.007" length="0.002"/>
+    </geometry>
+    <material name="grey">
+      <color rgba="0.5 0.5 0.5 1"/>
+    </material>
+  </visual>
+</link>
+<!-- Measuring Points -->
+<joint name="box_measuring_point_1_joint" type="fixed">
   <parent link="box_base_link"/>
-  <child link="box_socket_red"/>
-  <origin rpy="0 0 0" xyz="0 0 ${box_len_z}"/>
-</joint>
-<link name="box_socket_red">
-  <visual>
-    <origin rpy="0 0 0" xyz="0 0 0"/>
-    <geometry>
-      <cylinder radius="0.01" length="0.1"/>
-    </geometry>
-  </visual>
-</link>
-<joint name="box_socket_black_joint" type="fixed">
+  <child link="box_measuring_point_1"/>
+  <origin rpy="0 0 0" xyz="0 0 ${box_len_z}"/>
+</joint>
+<link name="box_measuring_point_1">
+  <visual>
+    <origin rpy="0 0 0" xyz="0 0 0"/>
+    <geometry>
+      <box size="0.01 0.01 0.1"/>
+    </geometry>
+  </visual>
+</link>
+<joint name="box_measuring_point_2_joint" type="fixed">
   <parent link="box_base_link"/>
-  <child link="box_socket_black"/>
-  <origin rpy="0 0 0" xyz="0 0 ${box_len_z}"/>
-</joint>
-<link name="box_socket_black">
-  <visual>
-    <origin rpy="0 0 0" xyz="0 0 0"/>
-    <geometry>
-      <cylinder radius="0.01" length="0.1"/>
-    </geometry>
-  </visual>
-</link>
-<joint name="box_socket_grey_joint" type="fixed">
-  <parent link="box_base_link"/>
-  <child link="box_socket_grey"/>
-  <origin rpy="0 0 0" xyz="0 0 ${box_len_z}"/>
-</joint>
-<link name="box_socket_grey">
-  <visual>
-    <origin rpy="0 0 0" xyz="0 0 0"/>
-    <geometry>
-      <cylinder radius="0.01" length="0.1"/>
-    </geometry>
-  </visual>
-</link>
-<!-- Clamping Strip -->
-<joint name="box_clamping_strip_1_joint" type="fixed">
-  <parent link="box_base_link"/>
-  <child link="box_clamping_strip_1"/>
-  <origin rpy="0 0 0" xyz="0 0 ${box_len_z}"/>
-</joint>
-<link name="box_clamping_strip_1">
+  <child link="box_measuring_point_2"/>
+  <origin rpy="0 0 0" xyz="0 0 ${box_len_z}"/>
+</joint>
+<link name="box_measuring_point_2">
   <visual>
     <origin rpy="0 0 0" xyz="0 0 0"/>
@@ -174,17 +206,53 @@
   </visual>
 </link>
-<joint name="box_clamping_strip_2_joint" type="fixed">
-  <parent link="box_base_link"/>
-  <child link="box_clamping_strip_2"/>
-  <origin rpy="0 0 0" xyz="0 0 ${box_len_z}"/>
-</joint>
-<link name="box_clamping_strip_2">
-  <visual>
-    <origin rpy="0 0 0" xyz="0 0 0"/>
-    <geometry>
-      <box size="0.01 0.01 0.1"/>
-    </geometry>
-  </visual>
-</link>
 <!-- Display -->
+<joint name="box_display_joint" type="fixed">
+  <parent link="box_corner_3"/>
+  <child link="box_display"/>
+  <origin rpy="0 0 0" xyz="-0.0545 -0.0325 ${box_len_z}"/>
+</joint>
+<link name="box_display">
+  <visual>
+    <origin rpy="0 0 ${pi/2}" xyz="0 0 ${0.0135/2}"/>
+    <geometry>
+      <box size="0.024 0.047 0.0135"/>
+    </geometry>
+    <material name="red">
+      <color rgba="1 0 0 1"/>
+    </material>
+  </visual>
+</link>
+<!-- Lid Handle -->
+<joint name="box_lid_handle_closed_joint" type="fixed">
+  <parent link="box_corner_4"/>
+  <child link="box_lid_handle_closed"/>
+  <origin rpy="0 0 0" xyz="0 0 ${box_len_z}"/>
+</joint>
+<link name="box_lid_handle_closed">
+  <visual>
+    <origin rpy="0 0 0" xyz="0 0 0"/>
+    <geometry>
+      <cylinder radius="0.01" length="0.01"/>
+    </geometry>
+    <material name="green">
+      <color rgba="0 1 0 1"/>
+    </material>
+  </visual>
+</link>
+<joint name="box_lid_handle_opened_joint" type="fixed">
+  <parent link="box_corner_4"/>
+  <child link="box_lid_handle_opened"/>
+  <origin rpy="0 0 0" xyz="0 0 ${box_len_z}"/>
+</joint>
+<link name="box_lid_handle_opened">
+  <visual>
+    <origin rpy="0 0 0" xyz="0 0 0"/>
+    <geometry>
+      <cylinder radius="0.01" length="0.01"/>
+    </geometry>
+    <material name="green">
+      <color rgba="0 1 0 1"/>
+    </material>
+  </visual>
+</link>
 </robot>

Commit message: edited box.urdf

File: box_description/urdf/box.urdf.xacro (robot description, xacro)
@@ -16,5 +16,5 @@
     <origin rpy="0 0 0" xyz="-${box_len_x/2} -${box_len_y/2} -${box_len_z/2}"/>
     <geometry>
-      <mesh filename="file:///media/jos/ExternalSSD/thi_robothix_grand_challenge/box_description/meshes/box.dae" scale="0.001 0.001 0.001"/>
+      <mesh filename="package://box_description/meshes/box.dae" scale="0.001 0.001 0.001"/>
     </geometry>
     <material name="white">
@@ -22,10 +22,4 @@
     </material>
   </visual>
-  <collision>
-    <origin rpy="0 0 0" xyz="-${box_len_x/2} -${box_len_y/2} -${box_len_z/2}"/>
-    <geometry>
-      <box size="-${box_len_x/2} -${box_len_y/2} -${box_len_z/2}}"/>
-    </geometry>
-  </collision>
 </link>
 <!-- Box Corners -->

Commit message: .urdf.xacro, moveit_interface.hpp, press_button.cpp edited, simulation is working, the robot goes to the definet frames.

File: box_description/urdf/box.urdf.xacro (robot description, xacro)
@@ -80,5 +80,5 @@
   <parent link="box_corner_2"/>
   <child link="box_button_blue"/>
-  <origin rpy="0 0 0" xyz="0.03405 -0.03225 ${box_len_z}"/>
+  <origin rpy="0 3.1416 3.1416" xyz="0.03405 -0.03225 ${box_len_z}"/>
 </joint>
 <link name="box_button_blue">
@@ -96,5 +96,5 @@
   <parent link="box_corner_2"/>
   <child link="box_button_red"/>
-  <origin rpy="0 0 0" xyz="0.04805 -0.03225 ${box_len_z}"/>
+  <origin rpy="0 3.1416 3.1416" xyz="0.04805 -0.03225 ${box_len_z}"/>
 </joint>
 <link name="box_button_red">
@@ -113,5 +113,5 @@
   <parent link="box_corner_3"/>
   <child link="box_slider"/>
-  <origin rpy="0 0 0" xyz="-0.0425 -0.0675 ${box_len_z}"/>
+  <origin rpy="0 3.1416 3.1416" xyz="-0.0425 -0.0675 ${box_len_z}"/>
   <limit effort="1000.0" lower="-0.0215" upper="0.0215" velocity="0.5"/>
 </joint>
@@ -128,5 +128,5 @@
   <parent link="box_corner_2"/>
   <child link="box_socket_red"/>
-  <origin rpy="0 0 0" xyz="0.0589 -0.0895 ${box_len_z}"/>
+  <origin rpy="0 3.1416 3.1416" xyz="0.0589 -0.0895 ${box_len_z}"/>
 </joint>
 <link name="box_socket_red">
@@ -144,5 +144,5 @@
   <parent link="box_corner_2"/>
   <child link="box_socket_black"/>
-  <origin rpy="0 0 0" xyz="0.034 -0.0895 ${box_len_z}"/>
+  <origin rpy="0 3.1416 3.1416" xyz="0.034 -0.0895 ${box_len_z}"/>
 </joint>
 <link name="box_socket_black">
@@ -221,5 +221,5 @@
   <parent link="box_corner_4"/>
   <child link="box_lid_handle_closed"/>
-  <origin rpy="0 0 0" xyz="0 0 ${box_len_z}"/>
+  <origin rpy="0 3.1416 3.1416" xyz="0 0 ${box_len_z}"/>
 </joint>
 <link name="box_lid_handle_closed">

Commit message: box.urdf.xacro edit opening positions added

File: box_description/urdf/box.urdf.xacro (robot description, xacro)
@@ -80,5 +80,5 @@
   <parent link="box_corner_2"/>
   <child link="box_button_blue"/>
-  <origin rpy="0 3.1416 3.1416" xyz="0.03405 -0.03225 ${box_len_z}"/>
+  <origin rpy="0 ${pi} ${pi}" xyz="0.03405 -0.03225 ${box_len_z}"/>
 </joint>
 <link name="box_button_blue">
@@ -96,5 +96,5 @@
   <parent link="box_corner_2"/>
   <child link="box_button_red"/>
-  <origin rpy="0 3.1416 3.1416" xyz="0.04805 -0.03225 ${box_len_z}"/>
+  <origin rpy="0 ${pi} ${pi}" xyz="0.04805 -0.03225 ${box_len_z}"/>
 </joint>
 <link name="box_button_red">
@@ -113,5 +113,5 @@
   <parent link="box_corner_3"/>
   <child link="box_slider"/>
-  <origin rpy="0 3.1416 3.1416" xyz="-0.0425 -0.0675 ${box_len_z}"/>
+  <origin rpy="0 ${pi} ${pi}" xyz="-0.0425 -0.0675 ${box_len_z}"/>
   <limit effort="1000.0" lower="-0.0215" upper="0.0215" velocity="0.5"/>
 </joint>
@@ -128,5 +128,5 @@
   <parent link="box_corner_2"/>
   <child link="box_socket_red"/>
-  <origin rpy="0 3.1416 3.1416" xyz="0.0589 -0.0895 ${box_len_z}"/>
+  <origin rpy="0 ${pi} ${pi}" xyz="0.0589 -0.0895 ${box_len_z}"/>
 </joint>
 <link name="box_socket_red">
@@ -144,5 +144,5 @@
   <parent link="box_corner_2"/>
   <child link="box_socket_black"/>
-  <origin rpy="0 3.1416 3.1416" xyz="0.034 -0.0895 ${box_len_z}"/>
+  <origin rpy="0 ${pi} ${pi}" xyz="0.034 -0.0895 ${box_len_z}"/>
 </joint>
 <link name="box_socket_black">
@@ -160,5 +160,5 @@
   <parent link="box_corner_4"/>
   <child link="box_socket_grey"/>
-  <origin rpy="0 -${pi/2} 0" xyz="-0.0482 0.0265 0.0963"/>
+  <origin rpy="0 -${pi/2} 0" xyz=" -0.0482 0.0265 0.0963"/>
 </joint>
 <link name="box_socket_grey">
@@ -177,5 +177,5 @@
   <parent link="box_base_link"/>
   <child link="box_measuring_point_1"/>
-  <origin rpy="0 0 0" xyz="0 0 ${box_len_z}"/>
+  <origin rpy="0 ${pi} ${pi}" xyz="0.0904 0.0836 0.072"/>
 </joint>
 <link name="box_measuring_point_1">
@@ -190,7 +190,20 @@
   <parent link="box_base_link"/>
   <child link="box_measuring_point_2"/>
-  <origin rpy="0 0 0" xyz="0 0 ${box_len_z}"/>
+  <origin rpy="0 ${pi} ${pi}" xyz="0.0528 0.0836 0.061"/>
 </joint>
 <link name="box_measuring_point_2">
+  <visual>
+    <origin rpy="0 0 0" xyz="0 0 0"/>
+    <geometry>
+      <box size="0.01 0.01 0.1"/>
+    </geometry>
+  </visual>
+</link>
+<joint name="box_measuring_point_3_joint" type="fixed">
+  <parent link="box_base_link"/>
+  <child link="box_measuring_point_3"/>
+  <origin rpy="0 ${pi} ${pi} " xyz="0.0394 0.0836 0.05"/>
+</joint>
+<link name="box_measuring_point_3">
   <visual>
     <origin rpy="0 0 0" xyz="0 0 0"/>
@@ -218,10 +231,10 @@
 </link>
 <!-- Lid Handle -->
-<joint name="box_lid_handle_closed_joint" type="fixed">
-  <parent link="box_corner_4"/>
-  <child link="box_lid_handle_closed"/>
-  <origin rpy="0 3.1416 3.1416" xyz="0 0 ${box_len_z}"/>
-</joint>
-<link name="box_lid_handle_closed">
+<joint name="box_lid_opening_pos_1_joint" type="fixed">
+  <parent link="box_corner_1"/>
+  <child link="box_lid_opening_pos_1"/>
+  <origin rpy="${pi} ${pi/2} ${-pi/2}" xyz="0.034 0.044 ${box_len_z}"/>
+</joint>
+<link name="box_lid_opening_pos_1">
   <visual>
     <origin rpy="0 0 0" xyz="0 0 0"/>
@@ -234,10 +247,10 @@
   </visual>
 </link>
-<joint name="box_lid_handle_opened_joint" type="fixed">
-  <parent link="box_corner_4"/>
-  <child link="box_lid_handle_opened"/>
-  <origin rpy="0 0 0" xyz="0 0 ${box_len_z}"/>
-</joint>
-<link name="box_lid_handle_opened">
+<joint name="box_lid_opening_pos_2_joint" type="fixed">
+  <parent link="box_corner_1"/>
+  <child link="box_lid_opening_pos_2"/>
+  <origin rpy="${pi} ${pi/2} ${-pi/2}" xyz="0.0955 0.044 ${box_len_z}"/>
+</joint>
+<link name="box_lid_opening_pos_2">
   <visual>
     <origin rpy="0 0 0" xyz="0 0 0"/>
@@ -250,3 +263,19 @@
   </visual>
 </link>
+<joint name="box_lid_opening_pos_3_joint" type="fixed">
+  <parent link="box_corner_1"/>
+  <child link="box_lid_opening_pos_3"/>
+  <origin rpy="${pi} ${pi/2} ${-pi/2}" xyz="0.0955 0.044 ${box_len_z + box_len_z}"/>
+</joint>
+<link name="box_lid_opening_pos_3">
+  <visual>
+    <origin rpy="0 0 0" xyz="0 0 0"/>
+    <geometry>
+      <cylinder radius="0.01" length="0.01"/>
+    </geometry>
+    <material name="green">
+      <color rgba="0 1 0 1"/>
+    </material>
+  </visual>
+</link>
 </robot>

Commit message: Slider start, middle and stop Frames defined

File: box_description/urdf/box.urdf.xacro (robot description, xacro)
@@ -110,10 +110,37 @@
 </link>
 <!-- Slider -->
-<joint name="box_slider_joint" type="fixed">
+<joint name="box_slider_joint_start" type="fixed">
   <parent link="box_corner_3"/>
-  <child link="box_slider"/>
-  <origin rpy="0 ${pi} ${pi}" xyz="-0.0425 -0.0675 ${box_len_z}"/>
-</joint>
-<link name="box_slider">
+  <child link="box_slider_start"/>
+  <!--Original x:-0.0425  y: -0.0675-->
+  <origin rpy="0 ${pi} ${pi}" xyz="-0.021 -0.0675 ${box_len_z}"/>
+</joint>
+<link name="box_slider_start">
+  <visual>
+    <origin rpy="0 0 0" xyz="0 0 0.005"/>
+    <geometry>
+      <box size="0.007 0.005796 0.01"/>
+    </geometry>
+  </visual>
+</link>
+<joint name="box_slider_joint_middle" type="fixed">
+  <parent link="box_corner_3"/>
+  <child link="box_slider_middle"/>
+  <origin rpy="0 ${pi} ${pi}" xyz="-0.0425 -0.0675  ${box_len_z}"/>
+</joint>
+<link name="box_slider_middle">
+  <visual>
+    <origin rpy="0 0 0" xyz="0 0 0.005"/>
+    <geometry>
+      <box size="0.007 0.005796 0.01"/>
+    </geometry>
+  </visual>
+</link>
+<joint name="box_slider_joint_stop" type="fixed">
+  <parent link="box_corner_3"/>
+  <child link="box_slider_stop"/>
+  <origin rpy="0 ${pi} ${pi}" xyz="-0.064 -0.0675 ${box_len_z}"/>
+</joint>
+<link name="box_slider_stop">
   <visual>
     <origin rpy="0 0 0" xyz="0 0 0.005"/>

Commit message: Added gripping point for probe

File: box_description/urdf/box.urdf.xacro (robot description, xacro)
@@ -186,7 +186,24 @@
   <parent link="box_corner_4"/>
   <child link="box_socket_grey"/>
-  <origin rpy="0 -${pi/2} 0" xyz=" -0.0482 0.0265 0.0963"/>
+  <origin rpy="${pi} -${pi/2} 0" xyz=" -0.0482 0.0265 0.0963"/>
 </joint>
 <link name="box_socket_grey">
+  <visual>
+    <origin rpy="0 0 0" xyz="0 0 -0.001"/>
+    <geometry>
+      <cylinder radius="0.007" length="0.002"/>
+    </geometry>
+    <material name="grey">
+      <color rgba="0.5 0.5 0.5 1"/>
+    </material>
+  </visual>
+</link>
+<!-- Probe gripping Point-->
+<joint name="box_probe_gripping_point_joint" type="fixed">
+  <parent link="box_corner_4"/>
+  <child link="box_probe_gripping_point"/>
+  <origin rpy="${pi} -${pi/2} 0" xyz=" -0.1488 0.0265 0.0963"/>
+</joint>
+<link name="box_probe_gripping_point">
   <visual>
     <origin rpy="0 0 0" xyz="0 0 -0.001"/>

Commit message: added probe gripping point and wrapping cable ponits

File: box_description/urdf/box.urdf.xacro (robot description, xacro)
@@ -203,5 +203,5 @@
   <parent link="box_corner_4"/>
   <child link="box_probe_gripping_point"/>
-  <origin rpy="${pi} -${pi/2} 0" xyz=" -0.1488 0.0265 0.0963"/>
+  <origin rpy="0 3.6128 ${pi}" xyz=" -0.1488 0.0265 0.0963"/>
 </joint>
 <link name="box_probe_gripping_point">
@@ -322,3 +322,52 @@
   </visual>
 </link>
+<!-- Cable wrapping Positions -->
+<joint name="box_cable_wrapping_pos_1_joint" type="fixed">
+  <parent link="box_corner_2"/>
+  <child link="box_cable_wrapping_pos_1"/>
+  <origin rpy="0 ${pi} ${pi}" xyz="0.0269 -0.0895 ${box_len_z + 0.005}"/>
+</joint>
+<link name="box_cable_wrapping_pos_1">
+  <visual>
+    <origin rpy="0 0 0" xyz="0 0 0.001"/>
+    <geometry>
+      <cylinder radius="0.007" length="0.002"/>
+    </geometry>
+    <material name="red">
+      <color rgba="1 0 0 1"/>
+    </material>
+  </visual>
+</link>
+<joint name="box_cable_wrapping_pos_2_joint" type="fixed">
+  <parent link="box_corner_2"/>
+  <child link="box_cable_wrapping_pos_2"/>
+  <origin rpy="0 ${pi} ${pi}" xyz="-0.02 -0.0895 ${box_len_z + 0.005}"/>
+</joint>
+<link name="box_cable_wrapping_pos_2">
+  <visual>
+    <origin rpy="0 0 0" xyz="0 0 0.001"/>
+    <geometry>
+      <cylinder radius="0.007" length="0.002"/>
+    </geometry>
+    <material name="red">
+      <color rgba="1 0 0 1"/>
+    </material>
+  </visual>
+</link>
+<joint name="box_cable_wrapping_pos_3_joint" type="fixed">
+  <parent link="box_corner_2"/>
+  <child link="box_cable_wrapping_pos_3"/>
+  <origin rpy="0 ${pi*(3/4)} ${pi}" xyz="-0.05 -0.0895 ${box_len_z - 0.02}"/>
+</joint>
+<link name="box_cable_wrapping_pos_3">
+  <visual>
+    <origin rpy="0 0 0" xyz="0 0 0.001"/>
+    <geometry>
+      <cylinder radius="0.007" length="0.002"/>
+    </geometry>
+    <material name="red">
+      <color rgba="1 0 0 1"/>
+    </material>
+  </visual>
+</link>
 </robot>

Commit message: prepared test

File: box_description/urdf/box.urdf.xacro (robot description, xacro)
@@ -150,4 +150,30 @@
   </visual>
 </link>
+<joint name="box_slider_joint_1" type="fixed">
+  <parent link="box_corner_3"/>
+  <child link="box_slider_1"/>
+  <origin rpy="0 ${pi} ${pi}" xyz="-0.03175 -0.0675 ${box_len_z}"/>
+</joint>
+<link name="box_slider_1">
+  <visual>
+    <origin rpy="0 0 0" xyz="0 0 0.005"/>
+    <geometry>
+      <box size="0.007 0.005796 0.01"/>
+    </geometry>
+  </visual>
+</link>
+<joint name="box_slider_joint_2" type="fixed">
+  <parent link="box_corner_3"/>
+  <child link="box_slider_2"/>
+  <origin rpy="0 ${pi} ${pi}" xyz="-0.05325 -0.0675 ${box_len_z}"/>
+</joint>
+<link name="box_slider_2">
+  <visual>
+    <origin rpy="0 0 0" xyz="0 0 0.005"/>
+    <geometry>
+      <box size="0.007 0.005796 0.01"/>
+    </geometry>
+  </visual>
+</link>
 <!-- Sockets -->
 <joint name="box_socket_red_joint" type="fixed">
